File: esp32_mcu_board/ESP32_MCU_Board.kicad_pcb (KiCad board)
At the start: 2 copper layers, 76.2 x 33 mm, 4 parts, among them J1 Conn_01x10, J2 Conn_01x10, J3 Conn_01x19, J4 Conn_01x19

Commit message: Added ESP32 MCU board to project description
Other:
- board text added: "ESP32-DevKitC-32E"
Changed lines of the file:
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@@
     (property "Sheetname" "")
     (attr through_hole)
-    (fp_text reference "J2" (at 3.302 0) (layer "B.SilkS")
-      (effects (font (size 1 1) (thickness 0.15)) (justify mirror))
+    (fp_text reference "J2" (at 0 3.175) (layer "F.SilkS")
+      (effects (font (size 1 1) (thickness 0.15)))
     )
     (fp_text value "Conn_01x10" (at 0 -25.63) (layer "B.Fab")
@@
     (property "Sheetname" "")
     (attr through_hole)
-    (fp_text reference "J1" (at -3.302 0) (layer "B.SilkS")
-      (effects (font (size 1 1) (thickness 0.15)) (justify mirror))
+    (fp_text reference "J1" (at 0 3.175) (layer "F.SilkS")
+      (effects (font (size 1 1) (thickness 0.15)))
     )
     (fp_text value "Conn_01x10" (at 0 -25.63) (layer "B.Fab")
@@
     (effects (font (size 1 1) (thickness 0.15)))
   )
+  (gr_text "ESP32-DevKitC-32E" (at 143.51 102.87) (layer "F.SilkS")
+    (effects (font (size 2 2) (thickness 0.3) italic))
+  )
   (gr_text "+5V" (at 167.64 111.125 90) (layer "F.SilkS")
     (effects (font (size 1 1) (thickness 0.15)))
@@
     (effects (font (size 1 1) (thickness 0.15)))
   )
+  (dimension (type aligned) (layer "F.SilkS")
+    (pts (xy 179.07 86.36) (xy 179.07 119.38))
+    (height -5.08)
+    (gr_text "33,0200 mm" (at 181.85 102.87 90) (layer "F.SilkS")
+      (effects (font (size 2 2) (thickness 0.3)))
+    )
+    (format (units 3) (units_format 1) (precision 4))
+    (style (thickness 0.15) (arrow_length 1.27) (text_position_mode 0) (extension_height 0.58642) (extension_offset 0.5) keep_text_aligned)
+  )
+  (dimension (type aligned) (layer "F.SilkS")
+    (pts (xy 101.6 120.65) (xy 177.8 120.65))
+    (height 5.08)
+    (gr_text "76,2000 mm" (at 139.7 123.43) (layer "F.SilkS")
+      (effects (font (size 2 2) (thickness 0.3)))
+    )
+    (format (units 3) (units_format 1) (precision 4))
+    (style (thickness 0.15) (arrow_length 1.27) (text_position_mode 0) (extension_height 0.58642) (extension_offset 0.5) keep_text_aligned)
+  )
 )

Commit message: Added ADS131M02IPWR ADC for MCU board to symbol and footprint library
Parts:
- added U1: ADS131M02IPWR, footprints:ADS131M02IPWR, F.Cu at (120.7, 102.2)
